File: RTD_Pi/RTD/RTD.kicad_pcb (KiCad board)
At the start: 2 copper layers, 7 parts, among them J1 Conn_01x08, J2 Conn_01x08, J3 Conn_01x08, J4 Conn_01x08, J5 Conn_01x08, J6 Conn_01x20, J7 Conn_01x08

Commit message: Some update
Parts:
- added C1: 10n, Capacitor_SMD:C_0603_1608Metric_Pad1.08x0.95mm_HandSolder, F.Cu at (128.6, 101.5)
- added C2: 10n, Capacitor_SMD:C_0603_1608Metric_Pad1.08x0.95mm_HandSolder, F.Cu at (149.6, 101.5)
Connections:
- net Net-(J1-Pin_4) renamed /GPIO 11
- net Net-(J1-Pin_5) renamed /GPIO 9
- net Net-(J1-Pin_6) renamed /GPIO 10
- net Net-(J1-Pin_7) renamed /GPIO 17
- net Net-(J2-Pin_7) renamed /GPIO 27
- net Net-(J3-Pin_7) renamed /GPIO 5
- net Net-(J4-Pin_7) renamed /GPIO 6
- net Net-(J5-Pin_7) renamed /GPIO 22
- net Net-(J6-Pin_2) renamed /GPIO 26
- J1 pad 1: Net-(J1-Pin_1) -> /3V3
- J1 pad 2: Net-(J1-Pin_2) -> /GND
- J2 pad 1: Net-(J1-Pin_1) -> /3V3
- J2 pad 2: Net-(J1-Pin_2) -> /GND
- J3 pad 1: Net-(J3-Pin_1) -> /3V3
- J3 pad 2: Net-(J3-Pin_2) -> /GND
- J4 pad 1: Net-(J3-Pin_1) -> /3V3
- J4 pad 2: Net-(J3-Pin_2) -> /GND
- J5 pad 1: Net-(J1-Pin_1) -> /3V3
- J5 pad 2: Net-(J1-Pin_2) -> /GND
- J6 pad 1: Net-(J1-Pin_1) -> /3V3
- J6 pad 13: Net-(J3-Pin_2) -> /GND
- J6 pad 14: unconnected-(J6-Pin_7-Pad14) -> /ID SD
- J6 pad 17: unconnected-(J6-Pin_4-Pad17) -> /GPIO 13
- J6 pad 18: unconnected-(J6-Pin_3-Pad18) -> /GPIO 19
- J6 pad 2: unconnected-(J6-Pin_19-Pad2) -> /GPIO 2
- J6 pad 20: unconnected-(J6-Pin_1-Pad20) -> /GND
- J6 pad 3: unconnected-(J6-Pin_18-Pad3) -> /GPIO 3
- J6 pad 4: unconnected-(J6-Pin_17-Pad4) -> /GPIO 4
- J6 pad 5: Net-(J1-Pin_2) -> /GND
- J6 pad 9: Net-(J3-Pin_1) -> /3V3
- J7 pad 1: Net-(J3-Pin_1) -> /3V3
- J7 pad 2: Net-(J3-Pin_2) -> /GND
Routing:
- net /GND: track 0.00 -> 132.9 mm
- net Net-(J3-Pin_2): track 93.9 -> 0.00 mm
- net /3V3: track 0.00 -> 65.3 mm, vias 0 -> 2
- net Net-(J3-Pin_1): track 28.7 -> 0.00 mm
- net Net-(J1-Pin_2): track 26.7 -> 0.00 mm
- net Net-(J1-Pin_1): track 23.5 -> 0.00 mm
- added copper zone on B.Cu, net /GND
- added copper zone on F.Cu, net /GND
Other:
- board outline added: 57.5 x 35 mm
