File: RTD_Pi/RTD/RTD.kicad_sch (KiCad schematic)
At the start: 7 parts, among them J1 Conn_01x08, J2 Conn_01x08, J3 Conn_01x08, J4 Conn_01x08, J5 Conn_01x08, J6 Conn_01x20, J7 Conn_01x08

Commit message: Some update
Parts:
- added C1, C2: 10n, Capacitor_SMD:C_0603_1608Metric_Pad1.08x0.95mm_HandSolder, symbol Device:C
Connections:
- net 3V3: now reaches J1.1 (Pin_1), J2.1 (Pin_1), J5.1 (Pin_1), J6.1 (Pin_20)
- net 3V3: now also J3.1 (Pin_1), J4.1 (Pin_1), J6.9 (Pin_12), J7.1 (Pin_1), C1.1, C2.1
- net GND: now reaches J1.2 (Pin_2), J2.2 (Pin_2), J5.2 (Pin_2), J6.5 (Pin_16)
- net GND: now also J3.2 (Pin_2), J4.2 (Pin_2), J6.13 (Pin_8), J6.20 (Pin_1), J7.2 (Pin_2), C1.2, C2.2
- net GPIO 11: now reaches J1.4 (Pin_4), J2.4 (Pin_4), J3.4 (Pin_4), J4.4 (Pin_4), J5.4 (Pin_4), J6.12 (Pin_9), J7.4 (Pin_4)
- net GPIO 9: now reaches J1.5 (Pin_5), J2.5 (Pin_5), J3.5 (Pin_5), J4.5 (Pin_5), J5.5 (Pin_5), J6.11 (Pin_10), J7.5 (Pin_5)
- net GPIO 10: now reaches J1.6 (Pin_6), J2.6 (Pin_6), J3.6 (Pin_6), J4.6 (Pin_6), J5.6 (Pin_6), J6.10 (Pin_11), J7.6 (Pin_6)
- net GPIO 27: now reaches J2.7 (Pin_7), J6.7 (Pin_14)
- net GPIO 6: now reaches J4.7 (Pin_7), J6.16 (Pin_5)
- net ID SD: now reaches J6.14 (Pin_7)
- net GPIO 5: now reaches J3.7 (Pin_7), J6.15 (Pin_6)
- net GPIO 13: now reaches J6.17 (Pin_4)
- net GPIO 19: now reaches J6.18 (Pin_3)
- net GPIO 26: now reaches J6.19 (Pin_2), J7.7 (Pin_7)
- net GPIO 2: now reaches J6.2 (Pin_19)
- net GPIO 3: now reaches J6.3 (Pin_18)
- net GPIO 4: now reaches J6.4 (Pin_17)
- net GPIO 17: now reaches J1.7 (Pin_7), J6.6 (Pin_15)
- net GPIO 22: now reaches J5.7 (Pin_7), J6.8
